File: PCB/FPGA_APU.sch (EAGLE design)
At the start: 140 parts, among them CON1 DIP40APU, U1 SN74LVC541A, U10 OPA2134U, U2 SN74LVC541A, U3 SN74LVC541A, U4 74LVC1G04GV, U5 74LVC4245APW,112, U6 EPCS4, U7 74LVC1G04GV, U8 EP2C5T144, U9 74LVC1G04GV, X1 057-010-1

Commit message: Add files via upload
Connections:
- net +3V3: no longer C11.P$2, C12.P$2, C13.P$2, U1.VCC, U2.VCC, U3.VCC
- net +5V: now also C11.P$2, C12.P$2, C13.P$2, U1.VCC, U2.VCC, U3.VCC
Changed lines of the file:
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@@
 <part name="V16" library="supply" deviceset="+3V3" device=""/>
 <part name="V17" library="supply" deviceset="+3V3" device=""/>
-<part name="V19" library="supply" deviceset="+3V3" device=""/>
 <part name="V20" library="supply" deviceset="+5V" device=""/>
 <part name="V21" library="supply" deviceset="+5V" device=""/>
@@
 <part name="GND8" library="supply1" library_urn="urn:adsk.eagle:library:371" deviceset="GND" device=""/>
 <part name="GND9" library="supply1" library_urn="urn:adsk.eagle:library:371" deviceset="GND" device=""/>
-<part name="V4" library="supply" deviceset="+3V3" device=""/>
 <part name="GND10" library="supply1" library_urn="urn:adsk.eagle:library:371" deviceset="GND" device=""/>
-<part name="V5" library="supply" deviceset="+3V3" device=""/>
 <part name="CON1" library="SnapEDA-Library" deviceset="DIP40APU" device=""/>
 <part name="GND11" library="supply1" library_urn="urn:adsk.eagle:library:371" deviceset="GND" device=""/>
@@
 <part name="C44" library="SnapEDA-Library" deviceset="CAP" device="" value="1nF"/>
 <part name="C45" library="SnapEDA-Library" deviceset="CAP" device="" value="1nF"/>
+<part name="V4" library="supply" deviceset="+5V" device=""/>
+<part name="V5" library="supply" deviceset="+5V" device=""/>
+<part name="V19" library="supply" deviceset="+5V" device=""/>
 </parts>
 <sheets>
@@
 <attribute name="VALUE" x="-123.87" y="89.665" size="1.778" layer="96" rot="R180"/>
 </instance>
-<instance part="V19" gate="G$1" x="-193.04" y="-17.78" smashed="yes" rot="R90">
-<attribute name="VALUE" x="-194.99" y="-17.015" size="1.778" layer="96" rot="R180"/>
-</instance>
 <instance part="V20" gate="1" x="-40.64" y="25.4" smashed="yes" rot="R270">
 <attribute name="VALUE" x="-38.75" y="24.59" size="1.778" layer="96"/>
@@
 <attribute name="VALUE" x="-187.96" y="15.24" size="1.778" layer="96"/>
 </instance>
-<instance part="V4" gate="G$1" x="-193.04" y="30.48" smashed="yes" rot="R90">
-<attribute name="VALUE" x="-194.99" y="31.245" size="1.778" layer="96" rot="R180"/>
-</instance>
 <instance part="GND10" gate="1" x="-185.42" y="66.04" smashed="yes">
 <attribute name="VALUE" x="-187.96" y="63.5" size="1.778" layer="96"/>
-</instance>
-<instance part="V5" gate="G$1" x="-193.04" y="78.74" smashed="yes" rot="R90">
-<attribute name="VALUE" x="-194.99" y="79.505" size="1.778" layer="96" rot="R180"/>
 </instance>
 <instance part="CON1" gate="G$1" x="-73.66" y="2.54" smashed="yes">
@@
 <attribute name="NAME" x="227.74" y="82.31" size="1.778" layer="95" rot="R180"/>
 <attribute name="VALUE" x="229.27" y="79.84" size="1.778" layer="96" rot="R180"/>
+</instance>
+<instance part="V4" gate="1" x="-193.04" y="-17.78" smashed="yes" rot="R90">
+<attribute name="VALUE" x="-194.93" y="-16.97" size="1.778" layer="96" rot="R180"/>
+</instance>
+<instance part="V5" gate="1" x="-193.04" y="30.48" smashed="yes" rot="R90">
+<attribute name="VALUE" x="-194.93" y="31.29" size="1.778" layer="96" rot="R180"/>
+</instance>
+<instance part="V19" gate="1" x="-193.04" y="78.74" smashed="yes" rot="R90">
+<attribute name="VALUE" x="-194.93" y="79.55" size="1.778" layer="96" rot="R180"/>
 </instance>
 </instances>
@@
 <junction x="-116.84" y="83.82"/>
 </segment>
+<segment>
+<wire x1="-190.5" y1="-17.78" x2="-185.42" y2="-17.78" width="0.1524" layer="91"/>
+<pinref part="U3" gate="G$1" pin="VCC"/>
+<pinref part="C13" gate="G$1" pin="P$2"/>
+<wire x1="-185.42" y1="-17.78" x2="-170.18" y2="-17.78" width="0.1524" layer="91"/>
+<junction x="-185.42" y="-17.78"/>
+<pinref part="V4" gate="1" pin="+5V"/>
+</segment>
+<segment>
+<wire x1="-190.5" y1="30.48" x2="-185.42" y2="30.48" width="0.1524" layer="91"/>
+<pinref part="U2" gate="G$1" pin="VCC"/>
+<pinref part="C12" gate="G$1" pin="P$2"/>
+<wire x1="-185.42" y1="30.48" x2="-170.18" y2="30.48" width="0.1524" layer="91"/>
+<junction x="-185.42" y="30.48"/>
+<pinref part="V5" gate="1" pin="+5V"/>
+</segment>
+<segment>
+<wire x1="-190.5" y1="78.74" x2="-185.42" y2="78.74" width="0.1524" layer="91"/>
+<pinref part="U1" gate="G$1" pin="VCC"/>
+<pinref part="C11" gate="G$1" pin="P$2"/>
+<wire x1="-185.42" y1="78.74" x2="-170.18" y2="78.74" width="0.1524" layer="91"/>
+<junction x="-185.42" y="78.74"/>
+<pinref part="V19" gate="1" pin="+5V"/>
+</segment>
 </net>
 <net name="+3V3" class="0">
@@
 </segment>
 <segment>
-<pinref part="V19" gate="G$1" pin="+3V3"/>
-<wire x1="-190.5" y1="-17.78" x2="-185.42" y2="-17.78" width="0.1524" layer="91"/>
-<pinref part="U3" gate="G$1" pin="VCC"/>
-<pinref part="C13" gate="G$1" pin="P$2"/>
-<wire x1="-185.42" y1="-17.78" x2="-170.18" y2="-17.78" width="0.1524" layer="91"/>
-<junction x="-185.42" y="-17.78"/>
-</segment>
-<segment>
-<pinref part="V4" gate="G$1" pin="+3V3"/>
-<wire x1="-190.5" y1="30.48" x2="-185.42" y2="30.48" width="0.1524" layer="91"/>
-<pinref part="U2" gate="G$1" pin="VCC"/>
-<pinref part="C12" gate="G$1" pin="P$2"/>
-<wire x1="-185.42" y1="30.48" x2="-170.18" y2="30.48" width="0.1524" layer="91"/>
-<junction x="-185.42" y="30.48"/>
-</segment>
-<segment>
-<pinref part="V5" gate="G$1" pin="+3V3"/>
-<wire x1="-190.5" y1="78.74" x2="-185.42" y2="78.74" width="0.1524" layer="91"/>
-<pinref part="U1" gate="G$1" pin="VCC"/>
-<pinref part="C11" gate="G$1" pin="P$2"/>
-<wire x1="-185.42" y1="78.74" x2="-170.18" y2="78.74" width="0.1524" layer="91"/>
-<junction x="-185.42" y="78.74"/>
-</segment>
-<segment>

Commit message: Add files via upload
Parts:
- U5: value 74LVC4245APW,112 -> SN74LVC8T245; device SnapEDA-Library:74LVC4245APW,112 -> SnapEDA-Library:SN74LVC8T245
Connections:
- net /OE: now also U5./OE; no longer U5.~OE
Changed lines of the file:
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@@
 <part name="U1" library="SnapEDA-Library" deviceset="SN74LVC541A" device=""/>
 <part name="U2" library="SnapEDA-Library" deviceset="SN74LVC541A" device=""/>
-<part name="U5" library="SnapEDA-Library" deviceset="74LVC4245APW,112" device=""/>
 <part name="GND8" library="supply1" library_urn="urn:adsk.eagle:library:371" deviceset="GND" device=""/>
 <part name="GND9" library="supply1" library_urn="urn:adsk.eagle:library:371" deviceset="GND" device=""/>
@@
 <part name="V5" library="supply" deviceset="+5V" device=""/>
 <part name="V19" library="supply" deviceset="+5V" device=""/>
+<part name="U5" library="SnapEDA-Library" deviceset="SN74LVC8T245" device=""/>
 </parts>
 <sheets>
@@
 <attribute name="VALUE" x="-162.56" y="20.32" size="1.778" layer="96"/>
 </instance>
-<instance part="U5" gate="A" x="-73.66" y="68.58" smashed="yes">
-<attribute name="NAME" x="-78.777040625" y="96.0745" size="2.08755" layer="95" ratio="10" rot="SR0"/>
-<attribute name="VALUE" x="-86.829790625" y="34.9687" size="2.08405" layer="96" ratio="10" rot="SR0"/>
-</instance>
 <instance part="GND8" gate="1" x="-175.26" y="73.66" smashed="yes" rot="R270">
 <attribute name="VALUE" x="-177.8" y="76.2" size="1.778" layer="96" rot="R270"/>
@@
 <instance part="V19" gate="1" x="-193.04" y="78.74" smashed="yes" rot="R90">
 <attribute name="VALUE" x="-194.93" y="79.55" size="1.778" layer="96" rot="R180"/>
+</instance>
+<instance part="U5" gate="G$1" x="-73.66" y="66.04" smashed="yes">
+<attribute name="NAME" x="-75.047040625" y="95.1545" size="2.08755" layer="95" ratio="10" rot="SR0"/>
+<attribute name="VALUE" x="-84.299790625" y="35.1387" size="2.08405" layer="96" ratio="10" rot="SR0"/>
 </instance>
 </instances>
@@
 <wire x1="-91.44" y1="43.18" x2="-96.52" y2="43.18" width="0.1524" layer="91"/>
 <junction x="-96.52" y="43.18"/>
-<pinref part="U5" gate="A" pin="GND@2"/>
-<pinref part="U5" gate="A" pin="GND@3"/>
-<pinref part="U5" gate="A" pin="GND@1"/>
+<pinref part="U5" gate="G$1" pin="GND@2"/>
+<pinref part="U5" gate="G$1" pin="GND@3"/>
+<pinref part="U5" gate="G$1" pin="GND@1"/>
 </segment>
 <segment>
@@
 <wire x1="-91.44" y1="78.74" x2="-106.68" y2="78.74" width="0.1524" layer="91"/>
 <label x="-106.68" y="78.74" size="1.778" layer="95"/>
-<pinref part="U5" gate="A" pin="DIR"/>
+<pinref part="U5" gate="G$1" pin="DIR"/>
 </segment>
 <segment>
@@
 <wire x1="-106.68" y1="76.2" x2="-91.44" y2="76.2" width="0.1524" layer="91"/>
 <label x="-106.68" y="76.2" size="1.778" layer="95"/>
-<pinref part="U5" gate="A" pin="~OE"/>
+<pinref part="U5" gate="G$1" pin="/OE"/>
 </segment>
 <segment>
@@
 <wire x1="-96.52" y1="86.36" x2="-91.44" y2="86.36" width="0.1524" layer="91"/>
 <wire x1="-91.44" y1="83.82" x2="-96.52" y2="83.82" width="0.1524" layer="91"/>
-<pinref part="U5" gate="A" pin="VCCB@2"/>
-<pinref part="U5" gate="A" pin="VCCB@1"/>
 <pinref part="V21" gate="1" pin="+5V"/>
 <wire x1="-96.52" y1="83.82" x2="-116.84" y2="83.82" width="0.1524" layer="91"/>
@@
 <wire x1="-116.84" y1="83.82" x2="-119.38" y2="83.82" width="0.1524" layer="91"/>
 <junction x="-116.84" y="83.82"/>
+<pinref part="U5" gate="G$1" pin="VCCB@2"/>
+<pinref part="U5" gate="G$1" pin="VCCB@1"/>
 </segment>
 <segment>
@@
 <wire x1="-119.38" y1="88.9" x2="-116.84" y2="88.9" width="0.1524" layer="91"/>
 <pinref part="V17" gate="G$1" pin="+3V3"/>
-<pinref part="U5" gate="A" pin="VCCA"/>
 <junction x="-116.84" y="88.9"/>
 <wire x1="-116.84" y1="88.9" x2="-91.44" y2="88.9" width="0.1524" layer="91"/>
+<pinref part="U5" gate="G$1" pin="VCCA"/>
 </segment>
 <segment>
@@
 </segment>
 <segment>
-<pinref part="U5" gate="A" pin="B7"/>
 <wire x1="-55.88" y1="71.12" x2="-43.18" y2="71.12" width="0.1524" layer="91"/>
 <label x="-53.34" y="71.12" size="1.778" layer="95"/>
+<pinref part="U5" gate="G$1" pin="B7"/>
 </segment>
 </net>
@@
 </segment>
 <segment>
-<pinref part="U5" gate="A" pin="B6"/>
 <wire x1="-55.88" y1="73.66" x2="-43.18" y2="73.66" width="0.1524" layer="91"/>
 <label x="-53.34" y="73.66" size="1.778" layer="95"/>
+<pinref part="U5" gate="G$1" pin="B6"/>
 </segment>
 </net>
@@
 </segment>
 <segment>
-<pinref part="U5" gate="A" pin="B5"/>
 <wire x1="-55.88" y1="76.2" x2="-43.18" y2="76.2" width="0.1524" layer="91"/>
 <label x="-53.34" y="76.2" size="1.778" layer="95"/>
+<pinref part="U5" gate="G$1" pin="B5"/>
 </segment>
 </net>
@@
 </segment>
 <segment>
-<pinref part="U5" gate="A" pin="B4"/>
 <wire x1="-55.88" y1="78.74" x2="-43.18" y2="78.74" width="0.1524" layer="91"/>
 <label x="-53.34" y="78.74" size="1.778" layer="95"/>
+<pinref part="U5" gate="G$1" pin="B4"/>
 </segment>
 </net>
@@
 </segment>
 <segment>
-<pinref part="U5" gate="A" pin="B3"/>
 <wire x1="-55.88" y1="81.28" x2="-43.18" y2="81.28" width="0.1524" layer="91"/>
 <label x="-53.34" y="81.28" size="1.778" layer="95"/>
+<pinref part="U5" gate="G$1" pin="B3"/>
 </segment>
 </net>
@@
 </segment>
 <segment>
-<pinref part="U5" gate="A" pin="B2"/>
 <wire x1="-55.88" y1="83.82" x2="-43.18" y2="83.82" width="0.1524" layer="91"/>
 <label x="-53.34" y="83.82" size="1.778" layer="95"/>
+<pinref part="U5" gate="G$1" pin="B2"/>
 </segment>
 </net>
@@
 </segment>
 <segment>
-<pinref part="U5" gate="A" pin="B1"/>
 <wire x1="-55.88" y1="86.36" x2="-43.18" y2="86.36" width="0.1524" layer="91"/>
 <label x="-53.34" y="86.36" size="1.778" layer="95"/>
+<pinref part="U5" gate="G$1" pin="B1"/>
 </segment>
 </net>
@@
 </segment>
 <segment>
-<pinref part="U5" gate="A" pin="B0"/>
 <wire x1="-55.88" y1="88.9" x2="-43.18" y2="88.9" width="0.1524" layer="91"/>
 <label x="-53.34" y="88.9" size="1.778" layer="95"/>
+<pinref part="U5" gate="G$1" pin="B0"/>
 </segment>
 </net>
@@
 <wire x1="-91.44" y1="71.12" x2="-106.68" y2="71.12" width="0.1524" layer="91"/>
 <label x="-106.68" y="71.12" size="1.778" layer="95"/>
-<pinref part="U5" gate="A" pin="A0"/>
+<pinref part="U5" gate="G$1" pin="A0"/>
 </segment>
 <segment>
@@
 <wire x1="-91.44" y1="68.58" x2="-106.68" y2="68.58" width="0.1524" layer="91"/>
 <label x="-106.68" y="68.58" size="1.778" layer="95"/>
-<pinref part="U5" gate="A" pin="A1"/>
+<pinref part="U5" gate="G$1" pin="A1"/>
 </segment>
 <segment>
@@
 <wire x1="-91.44" y1="66.04" x2="-106.68" y2="66.04" width="0.1524" layer="91"/>
 <label x="-106.68" y="66.04" size="1.778" layer="95"/>
-<pinref part="U5" gate="A" pin="A2"/>
+<pinref part="U5" gate="G$1" pin="A2"/>
 </segment>
 <segment>
@@
 <wire x1="-91.44" y1="53.34" x2="-106.68" y2="53.34" width="0.1524" layer="91"/>
 <label x="-106.68" y="53.34" size="1.778" layer="95"/>
-<pinref part="U5" gate="A" pin="A7"/>
+<pinref part="U5" gate="G$1" pin="A7"/>
 </segment>
 <segment>
@@
 <wire x1="-91.44" y1="55.88" x2="-106.68" y2="55.88" width="0.1524" layer="91"/>
 <label x="-106.68" y="55.88" size="1.778" layer="95"/>
-<pinref part="U5" gate="A" pin="A6"/>
+<pinref part="U5" gate="G$1" pin="A6"/>
 </segment>
 <segment>
@@
 <wire x1="-91.44" y1="58.42" x2="-106.68" y2="58.42" width="0.1524" layer="91"/>
 <label x="-106.68" y="58.42" size="1.778" layer="95"/>
-<pinref part="U5" gate="A" pin="A5"/>
+<pinref part="U5" gate="G$1" pin="A5"/>
 </segment>
 <segment>
@@
 <wire x1="-91.44" y1="60.96" x2="-106.68" y2="60.96" width="0.1524" layer="91"/>
 <label x="-106.68" y="60.96" size="1.778" layer="95"/>
-<pinref part="U5" gate="A" pin="A4"/>
+<pinref part="U5" gate="G$1" pin="A4"/>
 </segment>
 <segment>
@@
 <wire x1="-91.44" y1="63.5" x2="-106.68" y2="63.5" width="0.1524" layer="91"/>
 <label x="-106.68" y="63.5" size="1.778" layer="95"/>
-<pinref part="U5" gate="A" pin="A3"/>
-</segment>
-<segment>
+<pinref part="U5" gate="G$1" pin="A3"/>
+</segment>
+<segment>

Commit message: Add files via upload
Parts:
- C1, C6: value 22uF -> 0.1uF; device SnapEDA-Library:ELCAP -> rcl_my:C-EUC0805
- C10, C8: value 1uF -> 0.1uF; device SnapEDA-Library:CAP -> rcl_my:C-EUC0805
- C11, C13: value 0.1uF -> 1uF; device SnapEDA-Library:CAP -> rcl_my:C-EUC0805
- C12, C14, C15, C2, C26, C28, C29, C3, C30, C5, C7: device SnapEDA-Library:CAP -> rcl_my:C-EUC0805
- C16, C17, C18, C19, C20: value (none) -> 0.1uF; device SnapEDA-Library:CAP -> rcl_my:C-EUC0805
- C21, C22, C23, C24, C25: value 10uF -> 0.1uF; device SnapEDA-Library:CAP -> rcl_my:C-EUC0805
- C27: value 10uF -> 1uF; device SnapEDA-Library:CAP -> rcl_my:C-EUC0805
- C31: value 1uF -> (none); device SnapEDA-Library:CAP -> rcl_my:C-EUC0805
- C32, C33, C34, C35: value 0,1uF -> (none); device SnapEDA-Library:CAP -> rcl_my:C-EUC0805
- C36, C37, C38: value 0,1uF -> 1000; device SnapEDA-Library:CAP -> rcl_my:C-EUC0805
- C39, C40, C41, C42: value 0,1uF -> 10uF; device SnapEDA-Library:CAP -> rcl_my:C-EUC0805
- C4, C9: value 0.1uF -> 22uF; device SnapEDA-Library:CAP -> rcl_my:CPOL-EU153CLV-0505
- C43, C45: value 1nF -> 10uF; device SnapEDA-Library:CAP -> rcl_my:C-EUC0805
- C44: value 1nF -> 0.1uF; device SnapEDA-Library:CAP -> rcl_my:C-EUC0805
- R1: value 1k -> 75
- R11, R12, R13, R14, R15, R16, R17: value 1k -> (none)
- R18, R19, R20, R21, R22, R23, R24: value 2k -> (none)
- R2: value 1k -> 100
- R26, R28, R30: value 1k -> 2k
- R31, R33, R35, R48, R52: value 2k -> 1k
- R37, R39, R41, R43, R45, R53, R54, R56: value (none) -> 2k
- R38: value (none) -> 1.5k
- R4, R5: value 10k -> 1k
- R40, R42, R44, R46, R55: value (none) -> 1k
- R47: value 1.5k -> 2k
- R57, R58: value 10k -> 4.7k
- R61, R62: value 4.7k -> 510
- R63, R64: value 1 -> 1k
- R65, R66: value 510 -> 10k
- R67, R68: value 1k -> 1
- R7: value 100 -> 10k
- R8: value 75 -> 10k
Connections:
- removed net N$48: C25.P$2, R64.2
- removed net N$49: C45.P$1, JP3.1
- new net N$30: C42.1, R67.2
- new net N$37: C43.1, R68.2
- net +1V2: now also C27.1, C28.1, C29.1, C30.1, C8.1, C9.+; no longer C28.P$2, C29.P$2, C30.P$2, C31.P$2, C5.P$2
- net +3V3: now also C14.2, C37.1, C6.1, C7.1, R4.1, R8.2, R9.2; no longer C3.P$2, C4.P$2, C44.P$2, R2.1, R4.2, R5.2
- net +5V: now also C1.1, C15.1, C2.1, C3.1, C4.+, C41.1, C5.1, R57.1; no longer C11.P$2, C12.P$2, C13.P$2, C15.P$2, C2.P$2, C23.P$2, R65.1
- net CLK1: now also R2.2; no longer R7.2
- net CLK2: now also R1.2; no longer R8.2
- net DMC: now also R11.1; no longer R37.1
- net DMC0: now also R41.1; no longer R18.1
- net DMC1: now also R43.1; no longer R19.1
- net DMC2: now also R45.1; no longer R20.1
- net DMC3: now also R47.1; no longer R21.1
- net DMC4: now also R49.1; no longer R22.1
- net DMC5: now also R51.1; no longer R23.1
- net DMC6: now also R53.1; no longer R24.1
- net EXT_CLK: now also R2.1; no longer R7.1
- net GND: now also C10.2, C11.2, C12.2, C13.2, C36.2, C37.2, C4.-, C41.2, C44.1, C45.1, C5.2, C6.2, C7.2, C8.2, R25.1, R37.1, R40.1, R5.1, R56.2, R58.2, R7.2; no longer C43.P$1, C44.P$1, R1.1, R17.1, R30.1, R51.1, R52.2, R66.2, R9.2
- net N$1: now also R25.2, R26.2, R27.1; no longer R14.1, R15.2, R20.2
- net N$10: now also R30.2, R31.1; no longer R28.1, R32.2
- net N$11: now also C43.2; no longer C25.P$1
- net N$12: now also R32.2, R33.1; no longer R29.1, R30.2
- net N$13: now also R33.2, R34.2, R35.1; no longer R12.1, R13.2, R22.2
- net N$17: now also R40.2, R41.2, R42.1; no longer R13.1, R14.2, R21.2
- net N$18: now also R42.2, R43.2, R44.1; no longer R11.1, R12.2, R23.2
- net N$19: now also R52.2, R53.2, R54.2, R55.2, R56.1; no longer R11.2, R24.2, R49.2, R50.2, R52.1
- net N$2: now also C38.2, JP3.1; no longer C24.P$2, R63.2
- net N$20: now also R9.1; no longer R4.1
- net N$21: now also R8.1; no longer R5.1
- net N$23: now also R44.2, R45.2, R46.1; no longer R26.1, R27.2, R34.2
- net N$24: now also C36.1; no longer C43.P$2
- net N$25: now also R46.2, R47.2, R48.1; no longer R15.1, R16.2, R19.2
- net N$26: now also R48.2, R49.2, R50.1; no longer R25.1, R26.2, R35.2
- net N$27: now also R50.2, R51.2, R52.1; no longer R27.1, R28.2, R33.2
- net N$28: now also R38.2, R54.1; no longer R47.2, R49.1
- net N$29: now also R39.2, R55.1; no longer R48.2, R50.1
- net N$31: now also R35.2, R37.2, R38.1, R39.1; no longer R25.2, R47.1, R48.1, R51.2
- net N$32: now also C31.1, R11.2, R12.1; no longer C16.P$2, R37.2, R38.2
- net N$33: now also R12.2, R14.2, R16.2, R21.1, R22.1; no longer R38.1, R40.1, R42.1, R53.1, R54.1
- net N$34: now also C32.1, R13.2, R14.1; no longer C17.P$2, R39.2, R40.2
- net N$35: now also R18.2, R20.2, R23.2, R24.2; no longer R44.1, R46.1, R55.2, R56.2
- net N$36: now also C33.1, R15.2, R16.1; no longer C18.P$2, R41.2, R42.2
- net N$38: now also C34.1, R17.2, R18.1; no longer C19.P$2, R43.2, R44.2
- net N$39: now also R21.2, R23.1; no longer R53.2, R55.1
- net N$4: now also C42.2; no longer C24.P$1
- net N$40: now also C35.1, R19.2, R20.1; no longer C20.P$2, R45.2, R46.2
- net N$41: now also R22.2, R24.1; no longer R54.2, R56.1
- net N$42: now also R63.2, R65.1; no longer R57.1, R67.2
- net N$43: now also R65.2, R67.1; no longer R57.2, R63.1
- net N$44: now also R66.2, R68.1; no longer R58.2, R64.1
- net N$45: now also R64.2, R66.1; no longer R58.1, R68.2
- net N$46: now also C39.2, R57.2, R58.1; no longer C21.P$1, R59.2, R60.1
- net N$47: now also C40.2, R59.2, R60.1; no longer C22.P$1, R61.2, R62.1
- net N$6: now also C38.1, R1.1; no longer C45.P$2, R8.1
- net N$7: now also R7.1; no longer R9.1
- net N$9: now also R27.2, R28.2, R29.1; no longer R16.1, R17.2, R18.2
- net RND: now also R13.1; no longer R39.1
- net SND0: now also R26.1; no longer R31.1
- net SND1: now also R28.1; no longer R32.1
- net SND2: now also R30.1; no longer R33.1
- net SND3: now also R32.1; no longer R34.1
- net SND4: now also R34.1; no longer R35.1
- net SND_L: now also C39.1; no longer C21.P$2
- net SND_R: now also C40.1; no longer C22.P$2
- net SQA: now also R19.1; no longer R45.1
- net SQB: now also R17.1; no longer R43.1
- net TCK: now also R5.2; no longer R1.2
- net TMS: now also R4.2; no longer R2.2
- net TRIA: now also R15.1; no longer R41.1
- net VCC3.1: now also C16.1, C17.1, C18.1, C19.1, C20.1, C21.1, C22.1, C23.1, C24.1, C25.1, C26.1; no longer C32.P$2, C33.P$2, C34.P$2, C35.P$2, C36.P$2, C37.P$2, C38.P$2, C39.P$2, C40.P$2, C41.P$2, C42.P$2
- net VPPL1: now also C12.1, C13.1; no longer C7.P$2, C8.P$2
- net VPPL2: now also C10.1, C11.1; no longer C10.P$2, C9.P$2
- net VPPL3: now also C44.2, C45.2, R61.2, R62.1, R63.1, R64.1; no longer C26.P$2, C27.P$2, R65.2, R66.1, R67.1, R68.1
Other:
- moved on the sheet: C1, C6, R1, R11, R12, R13, R14, R15, R16, R17, R18, R19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

Commit message: Add files via upload
Parts:
- added C46: 10uF, rcl_my:C-EUC0805
- C42, C45: value 10uF -> 0.1uF
- C43: device rcl_my:C-EUC0805 -> rcl_my:CPOL-EU153CLV-0505
- C44: value 0.1uF -> 10uF; device rcl_my:C-EUC0805 -> rcl_my:CPOL-EU153CLV-0505
- R10: value 120 -> 160
- R25, R40: value 1k -> 2k
- renumbered CON1 to HEADER
Connections:
- new net N$48: C44.+, R68.2
- new net VPLL1: U8.PLL1_VCCA, U8.PLL1_VCCD
- net +5V: now also C42.2; no longer C4.+
- net GND: now also C45.2, C46.2; no longer C41.2, C44.1, C45.1
- net N$11: now also C44.-; no longer C43.2
- net N$30: now also C4.+; no longer C42.1, R67.2
- net N$37: now also C43.+, R67.2; no longer C43.1, R68.2
- net N$4: now also C43.-; no longer C42.2
- net VCC3.1: now also U8.VCCIO1@1, U8.VCCIO1@2, U8.VCCIO1@3, U8.VCCIO2@1, U8.VCCIO2@2, U8.VCCIO2@3, U8.VCCIO3@1, U8.VCCIO3@2, U8.VCCIO3@3, U8.VCCIO4@1, U8.VCCIO4@2, U8.VCCIO4@3; no longer U8.VCC@1, U8.VCC@10, U8.VCC@11, U8.VCC@12, U8.VCC@13, U8.VCC@15, U8.VCC@16, U8.VCC@18, U8.VCC@2, U8.VCC@20, U8.VCC@3, U8.VCC@5, U8.VCC@6, U8.VCC@8
- net VPPL1: no longer U8.VPLL1
- net VPPL2: now also U8.PLL2_VCCA, U8.PLL2_VCCD; no longer U8.VPLL2
- net VPPL3: now also C45.1, C46.1; no longer C44.2, C45.2
Other:
- moved on the sheet: C10, C11, C12, C13, C4, C42, C45, C7, C8, C9, L1, L2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
