File: PCB/V3/FPGA_APU V3.sch (EAGLE design)
At the start: 133 parts, among them U1 SN74LVC541A, U10 OPA2134U, U11 SN74LVC1G17DBVR, U2 SN74LVC541A, U3 SN74LVC541A, U4 74LVC1G04GV, U5 SN74LVC8T245, U6 EPCS4, U7 74LVC1G04GV, U8 EP2C5T144, U9 74LVC1G04GV, X1 057-010-1

Commit message: Add files via upload
Parts:
- removed U8: EP2C5T144, altera-cyclone-II:EP2C5T144
- added U15W: SN74LVC541A, SnapEDA-Library:SN74LVC541A
- C31, C32, C33, C34, C35: value (none) -> 0.01uF
- LED1: value (none) -> GNL-1206YC
- R11, R13, R15, R17, R19: value (none) -> 820
- R5: value 1k -> 10k
- R9: value 10k -> 1k
- U1: value SN74LVC541A -> EP2C5T144; device SnapEDA-Library:SN74LVC541A -> EP2C5T144:EP2C5T144
- X2: value (none) -> OUT
- XO1: value (none) -> 14.318MHz
- XO2: value (none) -> 17.73MHz
- renumbered Q1 to XO1, Q2 to XO2
Connections:
- removed net +1V2: C27.1, C28.1, C29.1, C30.1, C8.1, C9.+, L1.2, L2.1, U8.VCCINT@1, U8.VCCINT@2, U8.VCCINT@3, U8.VCCINT@4, VR2.VOUT
- removed net +3V3: C14.2, C37.1, C47.1, C6.1, C7.1, L3.1, R3.1, R37.2, R4.1, R6.2, R8.2, R9.2, U11.VCC, U5.VCCA, U6.VCC@1, U6.VCC@2, U6.VCC@3, VR1.VOUT, VR2.VIN, X1-4.S, XO2.VDD
- removed net DATAO: U6.ASDI, U8.DATA0
- removed net N$14: JP2-2.1, U8.IO30
- removed net N$15: JP2-3.1, U8.IO28
- removed net N$16: JP2-4.1, U8.IO27
- removed net N$20: R9.1, U8.NSTATUS
- removed net N$21: R8.1, U8.NCONFIG
- removed net N$22: R6.1, U8.CONF_DONE
- removed net N$30: C4.+
- removed net N$7: R7.1, U8.NCE
- removed net N$8 (its old number): JP2-1.1, U8.IO31
- removed net VCC3.1: C16.1, C17.1, C18.1, C19.1, C20.1, C21.1, C22.1, C23.1, C24.1, C25.1, C26.1, U8.VCCIO1@1, U8.VCCIO1@2, U8.VCCIO1@3, U8.VCCIO2@1, U8.VCCIO2@2, U8.VCCIO2@3, U8.VCCIO3@1, U8.VCCIO3@2, U8.VCCIO3@3, U8.VCCIO4@1, U8.VCCIO4@2, U8.VCCIO4@3
- removed net VPLL1: U8.PLL1_VCCA, U8.PLL1_VCCD
- new net CONF_DONE: R5.2, U1.CONF_DONE
- new net DATA0: U1.DATA0, U6.ASDI
- new net DENDY: JP2-2.1, U1.IO13
- new net J1: JP2-3.1, U1.IO12
- new net J2: JP2-4.1, U1.IO11
- new net N$1: RN4D.2, RN5D.1
- new net NCE: R8.1, U1.NCE
- new net NCONFIG: R7.1, U1.NCONFIG
- new net NSTATUS: R6.1, U1.NSTATUS
- new net NTSC/PAL: JP2-1.1, U1.IO14
- new net VCCINT: C27.2, C28.2, C29.1, C30.1, C8.1, C9.+, L1.2, L2.1, U1.VCCINT@1, U1.VCCINT@2, U1.VCCINT@3, U1.VCCINT@4, VR2.VOUT
- new net VCCIO: C14.2, C16.2, C17.2, C18.2, C19.2, C20.2, C21.2, C22.1, C23.1, C24.1, C25.1, C26.1, C37.1, C47.1, C6.1, C7.1, L3.1, R3.2, R37.2, R4.2, R5.1, R6.2, R7.2, U1.VCCIO1@1, U1.VCCIO1@2, U1.VCCIO1@3, U1.VCCIO2@1, U1.VCCIO2@2, U1.VCCIO2@3, U1.VCCIO3@1, U1.VCCIO3@2, U1.VCCIO3@3, U1.VCCIO4@1, U1.VCCIO4@2, U1.VCCIO4@3, U11.VCC, U4.VCC, U5.VCCA, U6.VCC@1, U6.VCC@2, U6.VCC@3, U7.VCC, U9.VCC, VR1.VOUT, VR2.VIN, X1-4.S, XO2.VDD
- net +5V: now also C15.2, C4.+, U15W.VCC; no longer C15.1, U1.VCC
- net /CSO: now also U1.IO2(/CSO); no longer U8.IO2(/CSO)
- net /IN0_FPGA: now also U1.IO72; no longer U8.IO133
- net /IN1_FPGA: now also U1.IO71; no longer U8.IO132
- net /OE: now also U1.IO55, U15W./OE1; no longer U1./OE1, U8.IO100
- net A0_FPGA: now also U1.IO58; no longer U8.IO104
- net A10: now also U15W.Y6; no longer U1.Y6
- net A10_FPGA: now also U1.IO75, U15W.A6; no longer U1.A6, U8.IO136
- net A11: now also U15W.Y5; no longer U1.Y5
- net A11_FPGA: now also U1.IO76, U15W.A5; no longer U1.A5, U8.IO137
- net A12: now also U15W.Y4; no longer U1.Y4
- net A12_FPGA: now also U1.IO77, U15W.A4; no longer U1.A4, U8.IO139
- net A13: now also U15W.Y3; no longer U1.Y3
- net A13_FPGA: now also U1.IO78, U15W.A3; no longer U1.A3, U8.IO141
- net A14: now also U15W.Y2; no longer U1.Y2
- net A14_FPGA: now also U1.IO79, U15W.A2; no longer U1.A2, U8.IO142
- net A15: now also U15W.Y1; no longer U1.Y1
- net A15_FPGA: now also U1.IO80, U15W.A1; no longer U1.A1, U8.IO143
- net A1_FPGA: now also U1.IO59; no longer U8.IO112
- net A2_FPGA: now also U1.IO60; no longer U8.IO113
- net A3_FPGA: now also U1.IO61; no longer U8.IO114
- net A4_FPGA: now also U1.IO62; no longer U8.IO115
- net A5_FPGA: now also U1.IO63; no longer U8.IO118
- net A6_FPGA: now also U1.IO64; no longer U8.IO119
- net A7_FPGA: now also U1.IO65; no longer U8.IO120
- net A8: now also U15W.Y8; no longer U1.Y8
- net A8_FPGA: now also U1.IO73, U15W.A8; no longer U1.A8, U8.IO134
- net A9: now also U15W.Y7; no longer U1.Y7
- net A9_FPGA: now also U1.IO74, U15W.A7; no longer U1.A7, U8.IO135
- net ASDO: now also U1.IO1(ASDO); no longer U8.IO1(ASDO)
- net CLK0: now also U1.CLK0; no longer U8.CLK0
- net CLK1: now also U1.CLK1; no longer U8.CLK1
- net CLK2: now also U1.CLK2; no longer U8.CLK2
- net DB0_FPGA: now also U1.IO3; no longer U8.IO3
- net DB1_FPGA: now also U1.IO4; no longer U8.IO4
- net DB2_FPGA: now also U1.IO5; no longer U8.IO7
- net DB3_FPGA: now also U1.IO6; no longer U8.IO8
- net DB4_FPGA: now also U1.IO7; no longer U8.IO9
- net DB5_FPGA: now also U1.IO8; no longer U8.IO24
- net DB6_FPGA: now also U1.IO9; no longer U8.IO25
- net DB7_FPGA: now also U1.IO10; no longer U8.IO26
- net DB_DIR: now also U1.IO81; no longer U8.IO144
- net DCLK: now also U1.DCLK; no longer U8.DCLK
- net DMC: now also U1.IO42; no longer U8.IO75
- net DMC0: now also U1.IO16; no longer U8.IO40
- net DMC1: now also U1.IO17; no longer U8.IO41
- net DMC2: now also U1.IO18; no longer U8.IO42
- net DMC3: now also U1.IO19; no longer U8.IO43
- net DMC4: now also U1.IO20; no longer U8.IO44
- net DMC5: now also U1.IO21; no longer U8.IO45
- net DMC6: now also U1.IO22; no longer U8.IO47
- net GND: now also C1.2, C15.1, C16.1, C17.1, C18.1, C19.1, C2.2, C20.1, C21.1, C22.2, C23.2, C24.2, C25.2, C26.2, C27.1, C28.1, C29.2, C3.2, C30.2, C31.2, C32.2, C33.2, C34.2, C35.2, C41.2, C47.2, C9.-, HEADER.DBG, R8.2, R9.2, U1.GAPLL1, U1.GAPLL2, U1.GND@1, U1.GND@10, U1.GND@11, U1.GND@12, U1.GND@13, U1.GND@14, U1.GND@18, U1.GND@19, U1.GND@2, U1.GND@20, U1.GND@21, U1.GND@22, U1.GND@23, U1.GND@3, U1.GND@7, U1.GND@8, U1.GND@9, U1.GPLL1@1, U1.GPLL1@2, U1.GPLL2@1, U1.GPLL2@2, U1.MSEL0, U1.MSEL1, U15W./OE2, U15W.GND, U4.GND, U7.GND, U9.GND, VR1.GND, VR2.GND; no longer R5.1, R7.2, U1./OE2, U1.GND, U8.GND@1, U8.GND@10, U8.GND@11, U8.GND@12, U8.GND@13, U8.GND@14, U8.GND@15, U8.GND@16, U8.GND@17, U8.GND@18, U8.GND@19, U8.GND@2, U8.GND@20, U8.GND@21, U8.GND@22, U8.GND@23, U8.GND@3, U8.GND@4, U8.GND@5, U8.GND@6, U8.GND@7, U8.GND@8, U8.GND@9, U8.MSEL0, U8.MSEL1
- net IRQ_FPGA: now also U1.IO57; no longer U8.IO103
- net M2_FPGA: now also U1.IO70; no longer U8.IO129
- net N$19: no longer RN4D.2, RN5D.1
- net NMI_FPGA: now also U1.IO56; no longer U8.IO101
- net OUT0_FPGA: now also U1.IO66; no longer U8.IO121
- net OUT1_FPGA: now also U1.IO67; no longer U8.IO122
- net OUT2_FPGA: now also U1.IO68; no longer U8.IO125
- net R/W_FPGA: now also U1.IO69; no longer U8.IO126
- net RES_FPGA: now also U1.IO54; no longer U8.IO99
- net RND: now also U1.IO43; no longer U8.IO76
- net SND0: now also U1.IO28; no longer U8.IO57
- net SND1: now also U1.IO27; no longer U8.IO55
- net SND2: now also U1.IO26; no longer U8.IO53
- net SND3: now also U1.IO25; no longer U8.IO52
- net SND4: now also U1.IO24; no longer U8.IO51
- net SND5: now also U1.IO23; no longer U8.IO48
- net SQA: now also U1.IO47; no longer U8.IO86
- net SQB: now also U1.IO46; no longer U8.IO81
- net TCK: now also R9.1, U1.TCK; no longer R5.2, U8.TCK
- net TDI: now also R3.1, U1.TDI; no longer R3.2, U8.TDI
- net TDO: now also U1.TDO; no longer U8.TDO
- net TMS: now also R4.1, U1.TMS; no longer R4.2, U8.TMS
- net TRIA: now also U1.IO45; no longer U8.IO80
- net VPPL1: now also U1.VAPLL1, U1.VPLL1
- net VPPL2: now also U1.VAPLL2, U1.VPLL2; no longer U8.PLL2_VCCA, U8.PLL2_VCCD
Other:
- moved on the sheet: C1, C10, C11, C12, C13, C14, C15, C16, C17, C18, C19, C2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

Commit message: Add files via upload
Parts:
- removed U15W: SN74LVC541A, SnapEDA-Library:SN74LVC541A
- added JP4: J2, jumper:JP4QE
- added JP8: DENDY, jumper:JP4QE
- added JP9: J1, jumper:JP4QE
- added U8: 74LVC1G04GV, 74LVC1G04GV:74LVC1G04GV
- C20, C22: value 0.1uF -> 1uF
- C27, C30: value 1uF -> 0.1uF
- C39, C40: value 10uF -> 0.1uF; device rcl_my:C-EUC0805 -> rcl_my:C-EUC0603
- C42: value 0.1uF -> 10uF
- C43: value 10uF -> 0.1uF; device rcl_my:CPOL-EU153CLV-0505 -> rcl_my:C-EUC0805
- C44: device rcl_my:CPOL-EU153CLV-0505 -> rcl_my:C-EUC0805
- C45: value 0.1uF -> 10uF; device rcl_my:C-EUC0805 -> rcl_my:CPOL-EU153CLV-0505
- C46: device rcl_my:C-EUC0805 -> rcl_my:CPOL-EU153CLV-0505
- C47: device rcl_my:C-EUC0603 -> rcl_my:C-EUC0805
- C48: value 0.1uF -> 10uF; device rcl_my:C-EUC0603 -> rcl_my:C-EUC0805
- JP2: value (none) -> NTSC/PAL
- R10: value 1k1 -> 820
- R11, R13, R15, R17, R19: value 820 -> (none)
- R12, R14, R16, R18: value (none) -> 820
- R2: value 75 -> 1k
- R24: value (none) -> 2k
- R27, R31, R34: value 2k -> 1k
- R28, R30, R35: value 1k -> 2k
- R29: value 1k -> 1.5k
- R32: value 1.5k -> 1k
- R36: value 2k -> 16k
- R37: value 16k -> 12k
- R38: value 12k -> 1k
- R39: value 1k -> 100
- R4: value 1k -> 10k
- R40: value 100 -> 75
- R8: value 10k -> 1k
- R9: value 1k -> 1k1
- U10: value OPA2134U -> EPCS4; device burr-brown:OPA2134U -> EPCS4:EPCS4
- U11: value SN74LVC1G17DBVR -> OPA2134U; device SN74LVC1G17DBVR:SN74LVC1G17DBVR -> burr-brown:OPA2134U
- U2: value SN74LVC541A -> 74LVC1G04GV; device SnapEDA-Library:SN74LVC541A -> 74LVC1G04GV:74LVC1G04GV
- U4: value 74LVC1G04GV -> SN74LVC541A; device 74LVC1G04GV:74LVC1G04GV -> SnapEDA-Library:SN74LVC541A
- U5: value SN74LVC8T245 -> SN74LVC541A; device SnapEDA-Library:SN74LVC8T245 -> SnapEDA-Library:SN74LVC541A
- U6: value EPCS4 -> 74LVC1G04GV; device EPCS4:EPCS4 -> 74LVC1G04GV:74LVC1G04GV
- U7: value 74LVC1G04GV -> SN74LVC8T245; device 74LVC1G04GV:74LVC1G04GV -> SnapEDA-Library:SN74LVC8T245
- U9: value 74LVC1G04GV -> SN74LVC1G17DBVR; device 74LVC1G04GV:74LVC1G04GV -> SN74LVC1G17DBVR:SN74LVC1G17DBVR
Connections:
- net +5V: now also C43.2, C44.1, R9.2, U11A.V+, U4.VCC, U5.VCC, U7.VCCB@1, U7.VCCB@2; no longer C41.1, C42.2, R10.2, U10A.V+, U15W.VCC, U2.VCC, U5.VCCB@1, U5.VCCB@2
- net /CSO: now also U10./CS; no longer U6./CS
- net /IN0: now also U5.Y5; no longer U3.Y5
- net /IN0_FPGA: now also U5.A5; no longer U3.A5
- net /IN1: now also U5.Y6; no longer U3.Y6
- net /IN1_FPGA: now also U5.A6; no longer U3.A6
- net /IRQ: now also U8.IN; no longer U9.IN
- net /NMI: now also U6.IN; no longer U7.IN
- net /OE: now also U3./OE1, U4./OE1, U5./OE2, U7./OE; no longer U15W./OE1, U2./OE1, U3./OE2, U5./OE
- net /RES: now also U2.IN; no longer U4.IN
- net A0: now also U4.Y8; no longer U2.Y8
- net A0_FPGA: now also U4.A8; no longer U2.A8
- net A1: now also U4.Y7; no longer U2.Y7
- net A10: now also U3.Y6; no longer U15W.Y6
- net A10_FPGA: now also U3.A6; no longer U15W.A6
- net A11: now also U3.Y5; no longer U15W.Y5
- net A11_FPGA: now also U3.A5; no longer U15W.A5
- net A12: now also U3.Y4; no longer U15W.Y4
- net A12_FPGA: now also U3.A4; no longer U15W.A4
- net A13: now also U3.Y3; no longer U15W.Y3
- net A13_FPGA: now also U3.A3; no longer U15W.A3
- net A14: now also U3.Y2; no longer U15W.Y2
- net A14_FPGA: now also U3.A2; no longer U15W.A2
- net A15: now also U3.Y1; no longer U15W.Y1
- net A15_FPGA: now also U3.A1; no longer U15W.A1
- net A1_FPGA: now also U4.A7; no longer U2.A7
- net A2: now also U4.Y6; no longer U2.Y6
- net A2_FPGA: now also U4.A6; no longer U2.A6
- net A3: now also U4.Y5; no longer U2.Y5
- net A3_FPGA: now also U4.A5; no longer U2.A5
- net A4: now also U4.Y4; no longer U2.Y4
- net A4_FPGA: now also U4.A4; no longer U2.A4
- net A5: now also U4.Y3; no longer U2.Y3
- net A5_FPGA: now also U4.A3; no longer U2.A3
- net A6: now also U4.Y2; no longer U2.Y2
- net A6_FPGA: now also U4.A2; no longer U2.A2
- net A7: now also U4.Y1; no longer U2.Y1
- net A7_FPGA: now also U4.A1; no longer U2.A1
- net A8: now also U3.Y8; no longer U15W.Y8
- net A8_FPGA: now also U3.A8; no longer U15W.A8
- net A9: now also U3.Y7; no longer U15W.Y7
- net A9_FPGA: now also U3.A7; no longer U15W.A7
- net ASDO: now also U10.DATA; no longer U6.DATA
- net CLK1: now also R39.2; no longer R40.2
- net CLK2: now also R40.2; no longer R2.2
- net CONF_DONE: now also R4.2; no longer R5.2
- net DATA0: now also U10.ASDI; no longer U6.ASDI
- net DB0: now also U7.B7; no longer U5.B7
- net DB0_FPGA: now also U7.A7; no longer U5.A7
- net DB1: now also U7.B6; no longer U5.B6
- net DB1_FPGA: now also U7.A6; no longer U5.A6
- net DB2: now also U7.B5; no longer U5.B5
- net DB2_FPGA: now also U7.A5; no longer U5.A5
- net DB3: now also U7.B4; no longer U5.B4
- net DB3_FPGA: now also U7.A4; no longer U5.A4
- net DB4: now also U7.B3; no longer U5.B3
- net DB4_FPGA: now also U7.A3; no longer U5.A3
- net DB5: now also U7.B2; no longer U5.B2
- net DB5_FPGA: now also U7.A2; no longer U5.A2
- net DB6: now also U7.B1; no longer U5.B1
- net DB6_FPGA: now also U7.A1; no longer U5.A1
- net DB7: now also U7.B0; no longer U5.B0
- net DB7_FPGA: now also U7.A0; no longer U5.A0
- net DB_DIR: now also U7.DIR; no longer U5.DIR
- net DCLK: now also U10.DCLK; no longer U6.DCLK
- net DENDY: now also JP8-1.1; no longer JP2-2.1
- net DMC: now also R10.1; no longer R11.1
- net EXT_CLK: now also R38.1, U9.A; no longer R39.1, U11.A
- net GND: now also C22.1, C23.1, C27.2, C28.2, C39.1, C40.2, C43.1, C44.2, C48.2, JP4-1.2, JP8-1.2, JP9-1.2, R24.1, R28.1, R35.2, R37.1, R7.2, U10.GND, U11A.V-, U3./OE2, U4./OE2, U5./OE1, U5.A1, U5.GND, U7.GND@1, U7.GND@2, U7.GND@3, U8.GND; no longer C22.2, C23.2, C27.1, C28.1, C41.2, C42.1, C45.2, C46.2, C48.1, JP2-2.2, JP2-3.2, JP2-4.2, R25.1, R31.1, R36.2, R38.1, R9.2, U10A.V-, U11.GND, U15W./OE2, U15W.GND, U2./OE2, U3./OE1, U3.A1, U5.GND@1, U5.GND@2, U5.GND@3, U7.GND
- net IRQ_FPGA: now also U8.OUT; no longer U9.OUT
- net J1: now also JP9-1.1; no longer JP2-3.1
- net J2: now also JP4-1.1; no longer JP2-4.1
- net M2: now also U5.Y8; no longer U3.Y8
- net M2_FPGA: now also U5.A8; no longer U3.A8
- net N$11: now also C46.-; no longer C44.-
- net N$18: now also R26.2, R27.1; no longer R27.2, R28.1
- net N$19: now also R33.2, R35.1; no longer R35.2, R36.1
- net N$27: now also R24.2, R27.2; no longer R26.2, R28.2
- net N$28: now also R29.2, R33.1; no longer R32.2, R34.1
- net N$29: now also R30.2, R34.1; no longer R33.2, R35.1
- net N$3: now also R28.2, R29.1, R30.1; no longer R31.2, R32.1, R33.1
- net N$32: now also R10.2, R11.1; no longer R11.2, R12.1
- net N$33: now also R11.2, R13.2, R15.2, R20.1; no longer R12.2, R14.2, R16.2, R22.1
- net N$34: now also R12.2, R13.1; no longer R13.2, R14.1
- net N$35: now also R17.2, R19.2, R22.2; no longer R18.2, R20.2, R24.2
- net N$36: now also R14.2, R15.1; no longer R15.2, R16.1
- net N$37: now also C45.+; no longer C43.+
- net N$38: now also R16.2, R17.1; no longer R17.2, R18.1
- net N$39: now also R20.2, R22.1; no longer R21.2, R23.1
- net N$4: now also C45.-; no longer C43.-
- net N$40: now also R18.2, R19.1; no longer R19.2, R20.1
- net N$41: now also R21.2, R23.1; no longer R22.2, R24.1
- net N$42: now also U11A.-IN; no longer U10A.-IN
- net N$43: now also U11A.OUT; no longer U10A.OUT
- net N$44: now also U11B.OUT; no longer U10B.OUT
- net N$46: now also C41.2, U11A.+IN; no longer C39.2, U10A.+IN
- net N$47: now also C42.2, U11B.+IN; no longer C40.2, U10B.+IN
- net N$48: now also C46.+; no longer C44.+
- net N$49: now also C39.2, R36.1, R37.2; no longer C48.2, R37.1, R39.2
- net N$5: now also R9.1; no longer R10.1
- net N$50: now also R39.1, U9.Y; no longer R40.1, U11.Y
- net N$53: now also R32.1; no longer R30.1
- net N$56: now also R31.2; no longer R29.2
- net N$57: now also R31.1, R32.2; no longer R29.1, R30.2
- net N$6: now also R40.1; no longer R2.1
- net N$8: now also U11B.-IN; no longer U10B.-IN
- net NCE: now also R7.1; no longer R8.1
- net NCONFIG: now also R6.1; no longer R7.1
- net NMI_FPGA: now also U6.OUT; no longer U7.OUT
- net NSTATUS: now also R5.1; no longer R6.1
- net OUT0: now also U5.Y2; no longer U3.Y2
- net OUT0_FPGA: now also U5.A2; no longer U3.A2
- net OUT1: now also U5.Y3; no longer U3.Y3
- net OUT1_FPGA: now also U5.A3; no longer U3.A3
- net OUT2: now also U5.Y4; no longer U3.Y4
- net OUT2_FPGA: now also U5.A4; no longer U3.A4
- net R/W: now also U5.Y7; no longer U3.Y7
- net R/W_FPGA: now also U5.A7; no longer U3.A7
- net RES_FPGA: now also U2.OUT; no longer U4.OUT
- net RND: now also R12.1; no longer R13.1
- net SND0: now also R25.1; no longer R26.1
- net SND1: now also R26.1; no longer R27.1
- net SND_L: now also C41.1; no longer C39.1
- net SND_R: now also C42.1; no longer C40.1
- net SQA: now also R18.1; no longer R19.1
- net SQB: now also R16.1; no longer R17.1
- net TCK: now also R8.1; no longer R9.1
- net TDI: now also R2.1; no longer R3.1
- net TMS: now also R3.1; no longer R4.1
- net TRIA: now also R14.1; no longer R15.1
- net VCCINT: now also C20.2, C22.2, C28.1; no longer C27.2, C28.2, C30.1
- net VCCIO: now also C23.2, C27.1, C30.1, C40.1, R2.2, R36.2, R4.1, R5.2, U10.VCC@1, U10.VCC@2, U10.VCC@3, U2.VCC, U6.VCC, U7.VCCA, U8.VCC; no longer C20.2, C22.1, C23.1, C47.1, R37.2, R4.2, R5.1, R7.2, U11.VCC, U4.VCC, U5.VCCA, U6.VCC@1, U6.VCC@2, U6.VCC@3, U7.VCC
- net VPPL3: now also C47.1, C48.1; no longer C45.1, C46.1
Other:
- note removed: "DENDY"
- note removed: "NTSC/PAL"
- moved on the sheet: C16, C17, C18, C19, C20, C21, C22, C23, C24, C25, C26, C27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
