File: PCB/V2/FPGA_APU.sch (EAGLE design)
At the start: 141 parts, among them U1 SN74LVC541A, U10 OPA2134U, U2 SN74LVC541A, U3 SN74LVC541A, U4 74LVC1G04GV, U5 SN74LVC8T245, U6 EPCS4, U7 74LVC1G04GV, U8 EP2C5T144, U9 74LVC1G04GV, X1 057-010-1

Commit message: Add files via upload
Parts:
- added JP4: J2, jumper:JP4QE
- added JP8: /DENDY, jumper:JP4QE
- added JP9: J1, jumper:JP4QE
- C31, C32, C33, C34, C35: value (none) -> 0.01uF
- JP2: value (none) -> /PAL
- LED1: value (none) -> GNL-1206YC
- R10: value 160 -> 1k2
- R11, R13, R15, R17, R19: value (none) -> 820
- X2: value (none) -> OUT
- XO1: value (none) -> 14.318MHz
- XO2: value (none) -> 17.734MHz
- renumbered Q1 to XO1, Q2 to XO2
Connections:
- net +1V2 renamed VCCINT
- removed net +3V3: C14.2, C37.1, C6.1, C7.1, L3.1, R3.1, R4.1, R6.2, R8.2, R9.2, U5.VCCA, U6.VCC@1, U6.VCC@2, U6.VCC@3, VR1.VOUT, VR2.VIN, X1-4.S, XO2.VDD
- removed net N$30: C4.+
- removed net VCC3.1: C16.1, C17.1, C18.1, C19.1, C20.1, C21.1, C22.1, C23.1, C24.1, C25.1, C26.1, U8.VCCIO1@1, U8.VCCIO1@2, U8.VCCIO1@3, U8.VCCIO2@1, U8.VCCIO2@2, U8.VCCIO2@3, U8.VCCIO3@1, U8.VCCIO3@2, U8.VCCIO3@3, U8.VCCIO4@1, U8.VCCIO4@2, U8.VCCIO4@3
- removed net VPPL1: C12.1, C13.1, L2.2
- new net VCCIO: C14.2, C16.1, C17.1, C18.1, C19.1, C20.1, C21.1, C22.1, C23.1, C24.1, C25.1, C26.1, C37.1, C6.1, C7.1, L3.1, R3.1, R4.1, R6.2, R8.2, R9.2, U4.VCC, U5.VCCA, U6.VCC@1, U6.VCC@2, U6.VCC@3, U7.VCC, U8.VCCIO1@1, U8.VCCIO1@2, U8.VCCIO1@3, U8.VCCIO2@1, U8.VCCIO2@2, U8.VCCIO2@3, U8.VCCIO3@1, U8.VCCIO3@2, U8.VCCIO3@3, U8.VCCIO4@1, U8.VCCIO4@2, U8.VCCIO4@3, U9.VCC, VR1.VOUT, VR2.VIN, X1-4.S, XO2.VDD
- net +5V: now also C15.2, C4.+; no longer C15.1
- net GND: now also C1.2, C14.1, C15.1, C16.2, C17.2, C18.2, C19.2, C2.2, C20.2, C21.2, C22.2, C23.2, C24.2, C25.2, C26.2, C27.2, C28.2, C29.2, C3.2, C30.2, C31.2, C32.2, C33.2, C34.2, C35.2, C41.2, C42.1, C9.-, HEADER.DBG, JP4-1.2, JP8-1.2, JP9-1.2, U4.GND, U7.GND, U9.GND, VR1.GND, VR2.GND; no longer JP2-2.2, JP2-3.2, JP2-4.2
- net N$14: now also JP8-1.1; no longer JP2-2.1
- net N$15: now also JP9-1.1; no longer JP2-3.1
- net N$16: now also JP4-1.1; no longer JP2-4.1
- net VPLL1: now also C12.1, C13.1, L2.2
Other:
- note removed: "DENDY"
- note removed: "NTSC/PAL"
- moved on the sheet: C1, C10, C11, C12, C13, C14, C15, C2, C3, C38, C4, C5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
